File: KiCAD/evo_ap/evo_ap.kicad_pcb (KiCad board)
At the start: 2 copper layers, 53.3 x 66 mm, 12 parts, among them J1 SN65HVD230_01x04, J2 RXB6, J3 Conn_01x02, J4 Conn_01x02, U1 ESP32-DEVKITC-32D, U2 TSR_1-2450

Commit message: Schema update using MCP2562
Other:
- board text removed: "CAN"
- board text removed: "GND"
- board text removed: "PROG"
- board text removed: "RADIO"
